Commit message: changed the world to jazzy compatible world, verified rqt graph for data movement

File: src/robot_sim/description/robot.urdf.xacro (robot description, xacro)
@@ -1,10 +1,6 @@
 <?xml version="1.0"?>
 <robot xmlns:xacro="http://www.ros.org/wiki/xacro" name="object_aware_robot">
-    <material name="white">
-        <color rgba="1 1 1 1"/>
-    </material>
-    <material name="blue">
-        <color rgba="0 0 1 1"/>
-    </material>
+    <material name="white"><color rgba="1 1 1 1"/></material>
+    <material name="blue"><color rgba="0 0 1 1"/></material>
     <link name="base_footprint"/>
     <joint name="base_footprint_joint" type="fixed">
@@ -16,14 +12,10 @@
         <visual>
             <origin xyz="0 0 0.075"/>
-            <geometry>
-                <box size="0.5 0.3 0.15"/>
-            </geometry>
+            <geometry><box size="0.5 0.3 0.15"/></geometry>
             <material name="white"/>
         </visual>
         <collision>
             <origin xyz="0 0 0.075"/>
-            <geometry>
-                <box size="0.5 0.3 0.15"/>
-            </geometry>
+            <geometry><box size="0.5 0.3 0.15"/></geometry>
         </collision>
         <inertial>
@@ -36,18 +28,14 @@
         <parent link="base_link"/>
         <child link="left_wheel"/>
-        <origin xyz="0 0.175 0" rpy="-${3.14159/2} 0 0"/>
+        <origin xyz="0 0.175 0" rpy="-1.570795 0 0"/>
         <axis xyz="0 0 1"/>
     </joint>
     <link name="left_wheel">
         <visual>
-            <geometry>
-                <cylinder radius="0.1" length="0.04"/>
-            </geometry>
+            <geometry><cylinder radius="0.1" length="0.04"/></geometry>
             <material name="blue"/>
         </visual>
         <collision>
-            <geometry>
-                <cylinder radius="0.1" length="0.04"/>
-            </geometry>
+            <geometry><cylinder radius="0.1" length="0.04"/></geometry>
         </collision>
         <inertial>
@@ -59,18 +47,14 @@
         <parent link="base_link"/>
         <child link="right_wheel"/>
-        <origin xyz="0 -0.175 0" rpy="${3.14159/2} 0 0"/>
+        <origin xyz="0 -0.175 0" rpy="1.570795 0 0"/>
         <axis xyz="0 0 1"/>
     </joint>
     <link name="right_wheel">
         <visual>
-            <geometry>
-                <cylinder radius="0.1" length="0.04"/>
-            </geometry>
+            <geometry><cylinder radius="0.1" length="0.04"/></geometry>
             <material name="blue"/>
         </visual>
         <collision>
-            <geometry>
-                <cylinder radius="0.1" length="0.04"/>
-            </geometry>
+            <geometry><cylinder radius="0.1" length="0.04"/></geometry>
         </collision>
         <inertial>
@@ -86,13 +70,9 @@
     <link name="caster_wheel">
         <visual>
-            <geometry>
-                <sphere radius="0.05"/>
-            </geometry>
+            <geometry><sphere radius="0.05"/></geometry>
             <material name="white"/>
         </visual>
         <collision>
-            <geometry>
-                <sphere radius="0.05"/>
-            </geometry>
+            <geometry><sphere radius="0.05"/></geometry>
         </collision>
         <inertial>
@@ -101,3 +81,119 @@
         </inertial>
     </link>
+    <joint name="laser_joint" type="fixed">
+        <parent link="base_link"/>
+        <child link="laser_frame"/>
+        <origin xyz="0.15 0 0.175" rpy="0 0 0"/>
+    </joint>
+    <link name="laser_frame">
+        <visual>
+            <geometry><cylinder radius="0.05" length="0.04"/></geometry>
+            <material name="blue"/>
+        </visual>
+        <collision>
+            <geometry><cylinder radius="0.05" length="0.04"/></geometry>
+        </collision>
+        <inertial>
+            <mass value="0.1"/>
+            <inertia ixx="0.000075" ixy="0.0" ixz="0.0" iyy="0.000075" iyz="0.0" izz="0.000125"/>
+        </inertial>
+    </link>
+    <joint name="camera_joint" type="fixed">
+        <parent link="base_link"/>
+        <child link="camera_link"/>
+        <origin xyz="0.25 0 0.1" rpy="0 0 0"/>
+    </joint>
+    <link name="camera_link">
+        <visual>
+            <geometry><box size="0.03 0.1 0.03"/></geometry>
+            <material name="blue"/>
+        </visual>
+        <collision>
+            <geometry><box size="0.03 0.1 0.03"/></geometry>
+        </collision>
+        <inertial>
+            <mass value="0.05"/>
+            <inertia ixx="0.000043" ixy="0.0" ixz="0.0" iyy="0.000008" iyz="0.0" izz="0.000043"/>
+        </inertial>
+    </link>
+    <gazebo reference="laser_joint"><preserveFixedJoint>true</preserveFixedJoint></gazebo>
+    <gazebo reference="camera_joint"><preserveFixedJoint>true</preserveFixedJoint></gazebo>
+    <gazebo reference="laser_frame">
+        <sensor type="gpu_ray" name="generic_lidar">
+            <pose>0 0 0 0 0 0</pose>
+            <topic>scan</topic>
+            <update_rate>10</update_rate>
+            <ray>
+                <scan>
+                    <horizontal>
+                        <samples>640</samples>
+                        <resolution>1</resolution>
+                        <min_angle>-3.14159</min_angle>
+                        <max_angle>3.14159</max_angle>
+                    </horizontal>
+                </scan>
+                <range>
+                    <min>0.15</min>
+                    <max>12.0</max>
+                    <resolution>0.01</resolution>
+                </range>
+            </ray>
+            <always_on>1</always_on>
+            <visualize>true</visualize>
+        </sensor>
+    </gazebo>
+    <gazebo reference="camera_link">
+        <sensor type="rgbd" name="generic_camera">
+            <pose>0 0 0 0 0 0</pose>
+            <topic>camera</topic>
+            <update_rate>30</update_rate>
+            <camera>
+                <horizontal_fov>1.089</horizontal_fov>
+                <image>
+                    <width>640</width>
+                    <height>480</height>
+                    <format>R8G8B8</format>
+                </image>
+                <clip>
+                    <near>0.05</near>
+                    <far>8.0</far>
+                </clip>
+            </camera>
+            <always_on>1</always_on>
+            <visualize>true</visualize>
+        </sensor>
+    </gazebo>
+    <gazebo reference="base_link">
+        <sensor type="imu" name="generic_imu">
+            <always_on>1</always_on>
+            <update_rate>100</update_rate>
+            <topic>imu/data</topic>
+        </sensor>
+    </gazebo>
+    <gazebo>
+        <plugin filename="gz-sim-odometry-publisher-system" name="gz::sim::systems::OdometryPublisher">
+            <dimensions>3</dimensions>
+            <odom_frame>odom</odom_frame>
+            <robot_base_frame>base_footprint</robot_base_frame> <odom_topic>odom</odom_topic>
+            <tf_topic>tf</tf_topic>
+        </plugin>
+    </gazebo>
+    <gazebo>
+        <plugin filename="gz-sim-diff-drive-system" name="gz::sim::systems::DiffDrive">
+            <left_joint>left_wheel_joint</left_joint>
+            <right_joint>right_wheel_joint</right_joint>
+            <wheel_separation>0.35</wheel_separation>
+            <wheel_diameter>0.2</wheel_diameter>
+            <max_wheel_torque>20</max_wheel_torque>
+            <max_wheel_acceleration>1.0</max_wheel_acceleration>
+            <odom_frame>odom</odom_frame>
+            <robot_base_frame>base_footprint</robot_base_frame>
+            <topic>/cmd_vel</topic>
+            <odom_topic>odom</odom_topic>
+            <tf_topic>tf</tf_topic>
+            <publish_odom>true</publish_odom>
+            <publish_odom_tf>false</publish_odom_tf>
+            <publish_wheel_tf>true</publish_wheel_tf>
+        </plugin>
+    </gazebo>
 </robot>
